File: Hardware/cloneduino_zero.kicad_pcb (KiCad board)
At the start: 4 copper layers, 50 x 19.6 mm, 34 parts, among them J1 USB-C Receptacle, J2 MicroSD Slot, J3 Conn_01x20, J4 Conn_01x20, J5 Conn_01x04, SW1 SW_Push, U1 SPX3819M5-L-3-3, U2 ATSAMD21G18A-A, Y1 32kHz

Commit message: Fix SD MOSI connection
Connections:
- J2 pad 3: /PA10 -> /PB10
Routing:
- net /PA10: track 29.1 -> 8.94 mm, vias 1 -> 0
- net /PB10: track 13.2 -> 29.1 mm, vias 0 -> 1
